Commit message: add gazebo configuration

File: urdf/titania.urdf.xacro (robot description, xacro)
@@ -15,10 +15,13 @@
     <xacro:property name="box_offset_rpy" value="0 0 0"/>
     <xacro:property name="fov_rad" value="${62.8 * pi/180.0}"/>
-    <xacro:property name="sim_w" value="320"/>
-    <xacro:property name="sim_h" value="240"/>
+    <xacro:property name="sim_w" value="752"/>
+    <xacro:property name="sim_h" value="480"/>
     <xacro:property name="sim_rate" value="1"/>
-    <xacro:property name="sim3d_w" value="320"/>
-    <xacro:property name="sim3d_h" value="240"/>
+    <xacro:property name="sim3d_w" value="752"/>
+    <xacro:property name="sim3d_h" value="480"/>
     <xacro:property name="sim3d_rate" value="0.1"/>
+    <material name="black">
+        <color rgba= "0.1 0.1 0.1 1.0"/>
+    </material>
     <link name="${camera_name}_cameraLeft_optical" />
     <link name="${camera_name}_cameraRight_optical" />
@@ -35,4 +38,15 @@
     <link name="${camera_name}_probe_mount"/>
     <link name="${camera_name}_center">
+        <pose>0 0 0 0 0 0</pose>
+        <inertial>
+            <mass value="5"/>
+            <origin rpy="0 0 0" xyz="0 0 0.1"/>
+            <inertia ixx="0.039" ixy="0" ixz="0" iyy="0.106" iyz="0" izz="0.0106"/>
+        </inertial>
+        <collision name="${camera_name}_center_collision">
+            <geometry>
+                <box size="${length} ${width} ${height}"/>
+            </geometry>
+        </collision>
         <visual>
             <xacro:if value="${(en_mesh == 'true')}">
@@ -51,7 +65,5 @@
             </geometry>
             <xacro:if value="${(en_mesh == 'false')}">
-                <material name="${camera_name}_camera_colour">
-                    <color rgba="0.1 0.1 0.1 1.0"/>
-                </material>
+                <material name="black"/>
             </xacro:if>
         </visual>
@@ -130,5 +142,5 @@
               <height>${sim_h}</height> <!-- real 480 -->
               <!-- <format>L8</format> -->
-              <format>R8G8B8</format>
+              <format>B8G8R8</format>
           </image>
           <clip>
@@ -144,56 +156,34 @@
     </xacro:macro>
     <gazebo reference="${camera_name}_cameraLeft">
-      <sensor type="multicamera" name="stereo_camera">
+      <sensor type="camera" name="camera_left">
         <update_rate>${sim_rate}</update_rate> <!-- reality 60fps on USB3-->
         <optical_camera name="left" />
-        <optical_camera name="right" />
-        <plugin name="stereo_camera_controller" filename="libgazebo_ros_multicamera.so">
+        <plugin name="camera_controller" filename="libgazebo_ros_camera.so">
           <alwaysOn>true</alwaysOn>
           <updateRate>${sim_rate}</updateRate>
-          <cameraName>${camera_name}</cameraName>
+          <cameraName>${camera_name}/left</cameraName>
           <imageTopicName>image_raw</imageTopicName>
           <cameraInfoTopicName>camera_info</cameraInfoTopicName>
           <frameName>${camera_name}_cameraLeft_optical</frameName>
-          <hackBaseline>0.07</hackBaseline>
-          <distortionK1>0.0</distortionK1>
-          <distortionK2>0.0</distortionK2>
-          <distortionK3>0.0</distortionK3>
-          <distortionT1>0.0</distortionT1>
-          <distortionT2>0.0</distortionT2>
         </plugin>
       </sensor>
     </gazebo>
-    <gazebo reference="${camera_name}_depth_optical_frame">
-      <sensor type="depth" name="${camera_name}_depth_camera">
-        <update_rate>${sim3d_rate}</update_rate>
-        <camera>
-          <horizontal_fov>${fov_rad}</horizontal_fov>
-          <image>
-            <format>B8G8R8</format>
-            <width>${sim3d_w}</width>
-            <height>${sim3d_h}</height>
-          </image>
-          <clip>
-            <near>0.05</near>
-            <far>5</far>
-          </clip>
-        </camera>
-        <plugin name="${camera_name}_depth_camera_controller" filename="libgazebo_ros_openni_kinect.so">
+    <gazebo reference="${camera_name}_cameraRight">
+      <sensor type="camera" name="camera_right">
+        <update_rate>${sim_rate}</update_rate> <!-- reality 60fps on USB3-->
+        <optical_camera name="right" />
+        <plugin name="camera_controller" filename="libgazebo_ros_camera.so">
           <alwaysOn>true</alwaysOn>
-          <updateRate>${sim3d_rate}</updateRate>
-          <frameName>${camera_name}_cameraLeft_optical</frameName>
-          <imageTopicName>${camera_name}_depth/image_raw</imageTopicName>
-          <cameraInfoTopicName>${camera_name}_depth/camera_info</cameraInfoTopicName>
-          <depthImageTopicName>${camera_name}_depth/depth/image_raw</depthImageTopicName>
-          <depthImageCameraInfoTopicName>${camera_name}_depth/depth/camera_info</depthImageCameraInfoTopicName>
-          <pointCloudTopicName>${camera_name}_depth/depth/points</pointCloudTopicName>
-          <distortion_k1>0.0</distortion_k1>
-          <distortion_k2>0.0</distortion_k2>
-          <distortion_k3>0.0</distortion_k3>
-          <distortion_t1>0.0</distortion_t1>
-          <distortion_t2>0.0</distortion_t2>
+          <updateRate>${sim_rate}</updateRate>
+          <cameraName>${camera_name}/right</cameraName>
+          <imageTopicName>image_raw</imageTopicName>
+          <cameraInfoTopicName>camera_info</cameraInfoTopicName>
+          <frameName>${camera_name}_cameraRight_optical</frameName>
         </plugin>
       </sensor>
     </gazebo>
+    <gazebo reference="${camera_name}_center">
+        <material>Gazebo/Black</material>
+    </gazebo>
   </xacro:macro>
 </robot>

Commit message: fix gazebo for generating stereo camera and add stl model

File: urdf/titania.urdf.xacro (robot description, xacro)
@@ -6,20 +6,20 @@
 <robot xmlns:xacro="http://ros.org/wiki/xacro">
     <xacro:macro name="titania_camera" params="camera_name:=titania en_mesh:=false en_imu:=false">
-    <xacro:property name="height" value="0.038"/>
-    <xacro:property name="width" value="0.10175"/>
-    <xacro:property name="length" value="0.03242"/>
+    <xacro:property name="height" value="0.059"/>
+    <xacro:property name="width" value="0.126"/>
+    <xacro:property name="length" value="0.0655"/>
+    <xacro:property name="baseline" value="0.09"/>
+    <xacro:property name="img_w" value="1600"/>
+    <xacro:property name="img_h" value="1600"/>
     <xacro:property name="mesh_file" value="package://i3dr_titania/mesh/titania.stl"/>
-    <xacro:property name="mesh_offset_xyz" value="-0.008 0.002 0"/>
-    <xacro:property name="mesh_offset_rpy" value="${pi/2} 0 ${pi/2}"/>
+    <xacro:property name="mesh_offset_xyz" value="0 0 -0.07"/>
+    <xacro:property name="mesh_offset_rpy" value="0 0 -${pi/2}"/>
     <xacro:property name="box_offset_xyz" value="0 0 0"/>
     <xacro:property name="box_offset_rpy" value="0 0 0"/>
-    <xacro:property name="fov_rad" value="${62.8 * pi/180.0}"/>
-    <xacro:property name="sim_w" value="752"/>
-    <xacro:property name="sim_h" value="480"/>
-    <xacro:property name="sim_rate" value="1"/>
-    <xacro:property name="sim3d_w" value="752"/>
-    <xacro:property name="sim3d_h" value="480"/>
-    <xacro:property name="sim3d_rate" value="0.1"/>
-    <material name="black">
+    <xacro:property name="fov_rad" value="${57.8 * pi/180.0}"/>
+    <xacro:property name="sim_w" value="${img_w/2}"/>
+    <xacro:property name="sim_h" value="${img_h/2}"/>
+    <xacro:property name="sim_rate" value="5"/>
+    <material name="darkgrey">
         <color rgba= "0.1 0.1 0.1 1.0"/>
     </material>
@@ -64,7 +64,5 @@
                 </xacro:if>
             </geometry>
-            <xacro:if value="${(en_mesh == 'false')}">
-                <material name="black"/>
-            </xacro:if>
+            <material name="darkgrey"/>
         </visual>
     </link>
@@ -91,10 +89,10 @@
         <parent link="${camera_name}_center"/>
         <child link="${camera_name}_cameraRight"/>
-        <origin xyz="0 ${-0.06/2}  0" rpy="0 0 0" />
+        <origin xyz="0 ${-baseline/2}  0" rpy="0 0 0" />
     </joint>
     <joint name="${camera_name}_left_camera_joint" type="fixed">
         <parent link="${camera_name}_center"/>
         <child link="${camera_name}_cameraLeft"/>
-        <origin xyz="0 ${0.06/2}  0" rpy="0 0 0" />
+        <origin xyz="0 ${baseline/2}  0" rpy="0 0 0" />
     </joint>
     <joint name="${camera_name}_left_optical_joint" type="fixed">
@@ -135,27 +133,49 @@
         <origin xyz="${(-0.03/2)-0.002} -0.007 ${-0.038/2}" rpy="0 0 0" />
     </joint>
-    <xacro:macro name="optical_camera" params="name fov_rad:=^ sim_w:=^ sim_h:=^">
+    <xacro:macro name="optical_camera" params="name offset fov_rad:=^ sim_w:=^ sim_h:=^">
         <camera name="${name}">
-          <horizontal_fov>${fov_rad}</horizontal_fov>
-          <image>
-              <width>${sim_w}</width> <!-- real: 752 -->
-              <height>${sim_h}</height> <!-- real 480 -->
-              <!-- <format>L8</format> -->
-              <format>B8G8R8</format>
-          </image>
-          <clip>
-              <near>0.02</near>
-              <far>300</far>
-          </clip>
-          <noise>
-              <type>gaussian</type>
-              <mean>0.0</mean>
-              <stddev>0.007</stddev>
-          </noise>
+            <pose>0 ${offset} 0 0 0 0</pose>
+            <horizontal_fov>${fov_rad}</horizontal_fov>
+            <image>
+                <width>${sim_w}</width>
+                <height>${sim_h}</height>
+                <format>B8G8R8</format>
+            </image>
+            <clip>
+                <near>0.02</near>
+                <far>300</far>
+            </clip>
+            <noise>
+                <type>gaussian</type>
+                <mean>0.0</mean>
+                <stddev>0.007</stddev>
+            </noise>
       </camera>
     </xacro:macro>
     <gazebo reference="${camera_name}_cameraLeft">
+      <sensor type="multicamera" name="stereo_camera">
+        <update_rate>${sim_rate}</update_rate> <!-- reality 60fps on USB3-->
+        <optical_camera name="left" offset="0" />
+        <optical_camera name="right" offset="${-baseline}" />
+        <plugin name="stereo_camera_controller" filename="libgazebo_ros_multicamera.so">
+          <alwaysOn>true</alwaysOn>
+          <updateRate>${sim_rate}</updateRate>
+          <cameraName>${camera_name}</cameraName>
+          <imageTopicName>image_raw</imageTopicName>
+          <cameraInfoTopicName>camera_info</cameraInfoTopicName>
+          <frameName>${camera_name}_cameraLeft_optical</frameName>
+          <!--<rightFrameName>${camera_name}_cameraRight_optical</rightFrameName>-->
+          <hackBaseline>${baseline}</hackBaseline>
+          <distortionK1>0.0</distortionK1>
+          <distortionK2>0.0</distortionK2>
+          <distortionK3>0.0</distortionK3>
+          <distortionT1>0.0</distortionT1>
+          <distortionT2>0.0</distortionT2>
+        </plugin>
+      </sensor>
+    </gazebo>
+    <!--<gazebo reference="${camera_name}_cameraLeft">
       <sensor type="camera" name="camera_left">
-        <update_rate>${sim_rate}</update_rate> <!-- reality 60fps on USB3-->
+        <update_rate>${sim_rate}</update_rate>
         <optical_camera name="left" />
         <plugin name="camera_controller" filename="libgazebo_ros_camera.so">
@@ -171,5 +191,5 @@
     <gazebo reference="${camera_name}_cameraRight">
       <sensor type="camera" name="camera_right">
-        <update_rate>${sim_rate}</update_rate> <!-- reality 60fps on USB3-->
+        <update_rate>${sim_rate}</update_rate>
         <optical_camera name="right" />
         <plugin name="camera_controller" filename="libgazebo_ros_camera.so">
@@ -183,6 +203,7 @@
       </sensor>
     </gazebo>
+    -->
     <gazebo reference="${camera_name}_center">
-        <material>Gazebo/Black</material>
+        <material>Gazebo/DarkGrey</material>
     </gazebo>
   </xacro:macro>

Commit message: fix image size in gazebo simulation

File: urdf/titania.urdf.xacro (robot description, xacro)
@@ -11,5 +11,5 @@
     <xacro:property name="baseline" value="0.09"/>
     <xacro:property name="img_w" value="1600"/>
-    <xacro:property name="img_h" value="1600"/>
+    <xacro:property name="img_h" value="1200"/>
     <xacro:property name="mesh_file" value="package://i3dr_titania/mesh/titania.stl"/>
     <xacro:property name="mesh_offset_xyz" value="0 0 -0.07"/>
@@ -20,5 +20,5 @@
     <xacro:property name="sim_w" value="${img_w/2}"/>
     <xacro:property name="sim_h" value="${img_h/2}"/>
-    <xacro:property name="sim_rate" value="5"/>
+    <xacro:property name="sim_rate" value="3"/>
     <material name="darkgrey">
         <color rgba= "0.1 0.1 0.1 1.0"/>
@@ -42,5 +42,5 @@
             <mass value="5"/>
             <origin rpy="0 0 0" xyz="0 0 0.1"/>
-            <inertia ixx="0.039" ixy="0" ixz="0" iyy="0.106" iyz="0" izz="0.0106"/>
+            <inertia ixx="0" ixy="0" ixz="0" iyy="0" iyz="0" izz="0"/>
         </inertial>
         <collision name="${camera_name}_center_collision">
@@ -69,10 +69,10 @@
     <xacro:if value="${(en_imu == 'true')}">
         <joint name="${camera_name}_imu_joint" type="fixed">
-            <origin xyz="0 0 0" rpy="${-pi/2} 0 ${-pi/2}" />
+            <origin xyz="0 0 0" rpy="0 0 0" />
             <parent link="${camera_name}_base_link" />
             <child link="${camera_name}_imu_link" />
         </joint>
         <joint name="${camera_name}_imu_mount_joint" type="fixed">
-            <origin xyz="0 0 0" rpy="${-pi/2} 0 ${-pi/2}" />
+            <origin xyz="0 0 0" rpy="0 0 0" />
             <parent link="${camera_name}_base_link" />
             <child link="${camera_name}_mount_base_link" />
@@ -89,10 +89,10 @@
         <parent link="${camera_name}_center"/>
         <child link="${camera_name}_cameraRight"/>
-        <origin xyz="0 ${-baseline/2}  0" rpy="0 0 0" />
+        <origin xyz="0.015 ${-baseline/2} 0" rpy="0 0 0" />
     </joint>
     <joint name="${camera_name}_left_camera_joint" type="fixed">
         <parent link="${camera_name}_center"/>
         <child link="${camera_name}_cameraLeft"/>
-        <origin xyz="0 ${baseline/2}  0" rpy="0 0 0" />
+        <origin xyz="0.015 ${baseline/2} 0" rpy="0 0 0" />
     </joint>
     <joint name="${camera_name}_left_optical_joint" type="fixed">
@@ -133,4 +133,5 @@
         <origin xyz="${(-0.03/2)-0.002} -0.007 ${-0.038/2}" rpy="0 0 0" />
     </joint>
+    <!-- Simulate stereo camera using gazebo -->
     <xacro:macro name="optical_camera" params="name offset fov_rad:=^ sim_w:=^ sim_h:=^">
         <camera name="${name}">
@@ -175,34 +176,30 @@
       </sensor>
     </gazebo>
-    <!--<gazebo reference="${camera_name}_cameraLeft">
-      <sensor type="camera" name="camera_left">
-        <update_rate>${sim_rate}</update_rate>
-        <optical_camera name="left" />
-        <plugin name="camera_controller" filename="libgazebo_ros_camera.so">
-          <alwaysOn>true</alwaysOn>
-          <updateRate>${sim_rate}</updateRate>
-          <cameraName>${camera_name}/left</cameraName>
-          <imageTopicName>image_raw</imageTopicName>
-          <cameraInfoTopicName>camera_info</cameraInfoTopicName>
-          <frameName>${camera_name}_cameraLeft_optical</frameName>
-        </plugin>
-      </sensor>
-    </gazebo>
-    <gazebo reference="${camera_name}_cameraRight">
-      <sensor type="camera" name="camera_right">
-        <update_rate>${sim_rate}</update_rate>
-        <optical_camera name="right" />
-        <plugin name="camera_controller" filename="libgazebo_ros_camera.so">
-          <alwaysOn>true</alwaysOn>
-          <updateRate>${sim_rate}</updateRate>
-          <cameraName>${camera_name}/right</cameraName>
-          <imageTopicName>image_raw</imageTopicName>
-          <cameraInfoTopicName>camera_info</cameraInfoTopicName>
-          <frameName>${camera_name}_cameraRight_optical</frameName>
-        </plugin>
-      </sensor>
-    </gazebo>
-    -->
+    <!-- Simulate IMU using gazebo -->
+    <xacro:if value="${(en_imu == 'true')}">
+        <gazebo reference="${camera_name}_imu_link">
+            <gravity>true</gravity>
+            <sensor name="imu_sensor" type="imu">
+            <always_on>true</always_on>
+            <update_rate>100</update_rate>
+            <visualize>true</visualize>
+            <topic>__default_topic__</topic>
+            <plugin filename="libgazebo_ros_imu_sensor.so" name="imu_plugin">
+                <topicName>imu</topicName>
+                <bodyName>${camera_name}_imu_link</bodyName>
+                <updateRateHZ>10.0</updateRateHZ>
+                <gaussianNoise>0.0</gaussianNoise>
+                <xyzOffset>0 0 0</xyzOffset>
+                <rpyOffset>0 0 0</rpyOffset>
+                <frameName>${camera_name}_imu_link</frameName>
+                <initialOrientationAsReference>false</initialOrientationAsReference>
+            </plugin>
+            <pose>0 0 0 0 0 0</pose>
+            </sensor>
+        </gazebo>
+    </xacro:if>
+    <!-- Attach material to gazebo object -->
     <gazebo reference="${camera_name}_center">
+        <gravity>0</gravity>
         <material>Gazebo/DarkGrey</material>
     </gazebo>

Commit message: simplify launchers

File: urdf/titania.urdf.xacro (robot description, xacro)
@@ -40,6 +40,6 @@
         <pose>0 0 0 0 0 0</pose>
         <inertial>
-            <mass value="5"/>
-            <origin rpy="0 0 0" xyz="0 0 0.1"/>
+            <mass value="0.5"/>
+            <origin rpy="0 0 0" xyz="0 0 0"/>
             <inertia ixx="0" ixy="0" ixz="0" iyy="0" iyz="0" izz="0"/>
         </inertial>
@@ -166,5 +166,4 @@
           <cameraInfoTopicName>camera_info</cameraInfoTopicName>
           <frameName>${camera_name}_cameraLeft_optical</frameName>
-          <!--<rightFrameName>${camera_name}_cameraRight_optical</rightFrameName>-->
           <hackBaseline>${baseline}</hackBaseline>
           <distortionK1>0.0</distortionK1>
@@ -201,5 +200,5 @@
     <!-- Attach material to gazebo object -->
     <gazebo reference="${camera_name}_center">
-        <gravity>0</gravity>
+        <gravity>true</gravity>
         <material>Gazebo/DarkGrey</material>
     </gazebo>

Commit message: add depth_min support

File: urdf/titania.urdf.xacro (robot description, xacro)
@@ -18,6 +18,6 @@
     <xacro:property name="box_offset_rpy" value="0 0 0"/>
     <xacro:property name="fov_rad" value="${57.8 * pi/180.0}"/>
-    <xacro:property name="sim_w" value="${img_w/2}"/>
-    <xacro:property name="sim_h" value="${img_h/2}"/>
+    <xacro:property name="sim_w" value="${img_w}/2"/>
+    <xacro:property name="sim_h" value="${img_h}/2"/>
     <xacro:property name="sim_rate" value="3"/>
     <material name="darkgrey">
@@ -40,5 +40,5 @@
         <pose>0 0 0 0 0 0</pose>
         <inertial>
-            <mass value="0.5"/>
+            <mass value="0.2"/>
             <origin rpy="0 0 0" xyz="0 0 0"/>
             <inertia ixx="0" ixy="0" ixz="0" iyy="0" iyz="0" izz="0"/>

Commit message: reduce mass in urdf

File: urdf/titania.urdf.xacro (robot description, xacro)
@@ -40,5 +40,5 @@
         <pose>0 0 0 0 0 0</pose>
         <inertial>
-            <mass value="0.2"/>
+            <mass value="0.15"/>
             <origin rpy="0 0 0" xyz="0 0 0"/>
             <inertia ixx="0" ixy="0" ixz="0" iyy="0" iyz="0" izz="0"/>

Commit message: remove downsampling resolution in urdf

File: urdf/titania.urdf.xacro (robot description, xacro)
@@ -18,6 +18,6 @@
     <xacro:property name="box_offset_rpy" value="0 0 0"/>
     <xacro:property name="fov_rad" value="${57.8 * pi/180.0}"/>
-    <xacro:property name="sim_w" value="${img_w}/2"/>
-    <xacro:property name="sim_h" value="${img_h}/2"/>
+    <xacro:property name="sim_w" value="${img_w}"/>
+    <xacro:property name="sim_h" value="${img_h}"/>
     <xacro:property name="sim_rate" value="3"/>
     <material name="darkgrey">

Commit message: update urdf

File: urdf/titania.urdf.xacro (robot description, xacro)
@@ -21,5 +21,5 @@
     <xacro:property name="sim_h" value="${img_h}"/>
     <xacro:property name="sim_rate" value="3"/>
-    <material name="darkgrey">
+    <material name="${camera_name}_darkgrey">
         <color rgba= "0.1 0.1 0.1 1.0"/>
     </material>
@@ -44,9 +44,9 @@
             <inertia ixx="0" ixy="0" ixz="0" iyy="0" iyz="0" izz="0"/>
         </inertial>
-        <collision name="${camera_name}_center_collision">
+        <!--<collision name="${camera_name}_center_collision">
             <geometry>
                 <box size="${length} ${width} ${height}"/>
             </geometry>
-        </collision>
+        </collision>-->
         <visual>
             <xacro:if value="${(en_mesh == 'true')}">
@@ -64,5 +64,5 @@
                 </xacro:if>
             </geometry>
-            <material name="darkgrey"/>
+            <material name="${camera_name}_darkgrey"/>
         </visual>
     </link>
@@ -80,5 +80,5 @@
     </xacro:if>
     <xacro:if value="${(en_imu == 'false')}">
-        <joint name="${camera_name}_imu_mount_joint" type="fixed">
+        <joint name="${camera_name}_base_mount_joint" type="fixed">
             <origin xyz="0 0 0" rpy="0 0 0" />
             <parent link="${camera_name}_base_link" />
@@ -116,5 +116,5 @@
         <parent link="${camera_name}_mount_base_link"/>
         <child link="${camera_name}_center"/>
-        <origin xyz="0 0 0" rpy="0 0 ${-pi/2}" />
+        <origin xyz="0 -0.0133 0.03" rpy="0 0 ${-pi/2}" />
     </joint>
     <joint name="${camera_name}_probe_mount_joint" type="fixed">
@@ -126,10 +126,10 @@
         <parent link="${camera_name}_mount_base_link"/>
         <child link="${camera_name}_mount_point_1"/>
-        <origin xyz="${(0.03/2)-0.002} -0.007 ${-0.038/2}" rpy="0 0 0" />
+        <origin xyz="${-0.025} -0 ${0}" rpy="0 0 0" />
     </joint>
     <joint name="${camera_name}_mount_point_2_joint" type="fixed">
         <parent link="${camera_name}_mount_base_link"/>
         <child link="${camera_name}_mount_point_2"/>
-        <origin xyz="${(-0.03/2)-0.002} -0.007 ${-0.038/2}" rpy="0 0 0" />
+        <origin xyz="${0.025} -0 ${0}" rpy="0 0 0" />
     </joint>
     <!-- Simulate stereo camera using gazebo -->

Commit message: fix urdf

File: urdf/titania.urdf.xacro (robot description, xacro)
@@ -13,5 +13,5 @@
     <xacro:property name="img_h" value="1200"/>
     <xacro:property name="mesh_file" value="package://i3dr_titania/mesh/titania.stl"/>
-    <xacro:property name="mesh_offset_xyz" value="0 0 -0.07"/>
+    <xacro:property name="mesh_offset_xyz" value="0 0 -0.072"/>
     <xacro:property name="mesh_offset_rpy" value="0 0 -${pi/2}"/>
     <xacro:property name="box_offset_xyz" value="0 0 0"/>
@@ -116,5 +116,5 @@
         <parent link="${camera_name}_mount_base_link"/>
         <child link="${camera_name}_center"/>
-        <origin xyz="0 -0.0133 0.03" rpy="0 0 ${-pi/2}" />
+        <origin xyz="0 -0.0133 0.0315" rpy="0 0 ${-pi/2}" />
     </joint>
     <joint name="${camera_name}_probe_mount_joint" type="fixed">
