Commit message: add optional collision for urdf

File: urdf/titania.urdf.xacro (robot description, xacro)
@@ -5,5 +5,5 @@
 -->
 <robot xmlns:xacro="http://wiki.ros.org/xacro">
-    <xacro:macro name="titania_camera" params="camera_name:=titania en_mesh:=false en_imu:=false">
+    <xacro:macro name="titania_camera" params="camera_name:=titania en_mesh:=false en_imu:=false en_collision:=true">
     <xacro:property name="height" value="0.059"/>
     <xacro:property name="width" value="0.126"/>
@@ -44,9 +44,11 @@
             <inertia ixx="0" ixy="0" ixz="0" iyy="0" iyz="0" izz="0"/>
         </inertial>
-        <!--<collision name="${camera_name}_center_collision">
-            <geometry>
-                <box size="${length} ${width} ${height}"/>
-            </geometry>
-        </collision>-->
+        <xacro:if value="${(en_collision == 'true')}">
+            <collision name="${camera_name}_center_collision">
+                <geometry>
+                    <box size="${length} ${width} ${height}"/>
+                </geometry>
+            </collision>
+        </xacro:if>
         <visual>
             <xacro:if value="${(en_mesh == 'true')}">
@@ -89,10 +91,10 @@
         <parent link="${camera_name}_center"/>
         <child link="${camera_name}_cameraRight"/>
-        <origin xyz="0.015 ${-baseline/2} 0" rpy="0 0 0" />
+        <origin xyz="0.015 ${(-baseline/2)+0.002} 0" rpy="0 0 0" />
     </joint>
     <joint name="${camera_name}_left_camera_joint" type="fixed">
         <parent link="${camera_name}_center"/>
         <child link="${camera_name}_cameraLeft"/>
-        <origin xyz="0.015 ${baseline/2} 0" rpy="0 0 0" />
+        <origin xyz="0.015 ${(baseline/2)+0.002} 0" rpy="0 0 0" />
     </joint>
     <joint name="${camera_name}_left_optical_joint" type="fixed">

File: urdf/titania_scene.urdf.xacro (robot description, xacro)
@@ -8,5 +8,6 @@
     <xacro:arg name="en_imu" default="false"/>
     <xacro:arg name="en_mesh" default="false"/>
+    <xacro:arg name="en_collision" default="true"/>
     <xacro:include filename="$(find i3dr_titania)/urdf/titania.urdf.xacro" />
-    <xacro:titania_camera camera_name="$(arg camera_name)" en_mesh="$(arg en_mesh)" en_imu="$(arg en_imu)"/>
+    <xacro:titania_camera camera_name="$(arg camera_name)" en_collision="$(arg en_collision)" en_mesh="$(arg en_mesh)" en_imu="$(arg en_imu)"/>
 </robot>
